File: circuit/bird.brd (EAGLE design)
At the start: 42.1 x 37.9 mm, 24 parts, among them J1 22-27-2031-03, U1 ATTINY84-20SSU, X1 MINI-USB-32005-201

Commit message: cleanups and fix sketch
Parts:
- added TP1: TEST-POINT2, SparkFun:PAD.02X.02
Connections:
- net MAGNETIC_REFERENCE: now also TP1.P$1
Routing:
- net MAGNETIC_REFERENCE: track 0.00 -> 4.74 mm
- net 5V: track 166.4 -> 167.8 mm
Changed lines of the file:
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@@
 <grid distance="0.1" unitdist="mm" unit="mm" style="lines" multiple="1" display="yes" altdistance="0.001" altunitdist="mm" altunit="mm"/>
 <layers>
-<layer number="1" name="Top" color="4" fill="1" visible="no" active="yes"/>
+<layer number="1" name="Top" color="4" fill="1" visible="yes" active="yes"/>
 <layer number="2" name="Route2" color="1" fill="3" visible="no" active="no"/>
 <layer number="3" name="Route3" color="4" fill="3" visible="no" active="no"/>
 <layer number="14" name="Route14" color="1" fill="6" visible="no" active="no"/>
 <layer number="15" name="Route15" color="4" fill="6" visible="no" active="no"/>
-<layer number="16" name="Bottom" color="1" fill="1" visible="no" active="yes"/>
+<layer number="16" name="Bottom" color="1" fill="1" visible="yes" active="yes"/>
 <layer number="17" name="Pads" color="2" fill="1" visible="yes" active="yes"/>
 <layer number="18" name="Vias" color="2" fill="1" visible="yes" active="yes"/>
@@
 <attribute name="NAME" x="4.485" y="1.055" size="1.27" layer="25" rot="R90"/>
 </element>
+<element name="TP1" library="SparkFun" package="PAD.02X.02" value="TEST-POINT2" x="29.7" y="11.7"/>
 </elements>
 <signals>
@@
 <wire x1="14.9352" y1="14.6304" x2="14.9079" y2="14.7696" width="0.254" layer="1"/>
 <wire x1="17.3736" y1="9.144" x2="17.6" y2="8.94" width="0.254" layer="1"/>
-<wire x1="25.6032" y1="2.7432" x2="28.3464" y2="5.4864" width="0.254" layer="1"/>
-<wire x1="28.3464" y1="5.4864" x2="30.1752" y2="7.3152" width="0.254" layer="1"/>
+<wire x1="25.6032" y1="2.7432" x2="31.0974" y2="8.1544" width="0.254" layer="1"/>
+<wire x1="31.0974" y1="8.1544" x2="30.1752" y2="7.3152" width="0.254" layer="1"/>
 <wire x1="30.1752" y1="7.3152" x2="30.21" y2="7.35" width="0.254" layer="1"/>
 <wire x1="25.6032" y1="2.7432" x2="25.5" y2="2.685" width="0.254" layer="1"/>
 <wire x1="28.3464" y1="16.1544" x2="28.6512" y2="16.4592" width="0.254" layer="1"/>
 <wire x1="28.6512" y1="16.4592" x2="30.1752" y2="17.9832" width="0.254" layer="1"/>
-<wire x1="28.3464" y1="5.4864" x2="28.3464" y2="16.1544" width="0.254" layer="1"/>
+<wire x1="31.0974" y1="8.1544" x2="31.1" y2="12.3" width="0.254" layer="1"/>
+<wire x1="31.1" y1="12.3" x2="28.366" y2="14.0074" width="0.254" layer="1"/>
+<wire x1="28.366" y1="14.0074" x2="28.3464" y2="16.1544" width="0.254" layer="1"/>
 <wire x1="30.1752" y1="17.9832" x2="30.31" y2="18.08" width="0.254" layer="1"/>
 <wire x1="19.2024" y1="7.3152" x2="17.6784" y2="8.8392" width="0.254" layer="1"/>
@@
 <signal name="MAGNETIC_REFERENCE">
 <contactref element="U1" pad="10"/>
+<contactref element="TP1" pad="P$1"/>
+<wire x1="29.7" y1="11.7" x2="28.8" y2="11.7" width="0.254" layer="1"/>
+<wire x1="28.8" y1="11.7" x2="27.5" y2="13" width="0.254" layer="1"/>
+<wire x1="27.5" y1="13" x2="25.5938" y2="13" width="0.254" layer="1"/>
+<wire x1="25.5938" y1="13" x2="25.5238" y2="12.93" width="0.254" layer="1"/>
 </signal>
 <signal name="ROLL_SERVO">

Commit message: ground
Routing:
- net GND: track 134.4 -> 132.6 mm, vias 2 -> 4
Changed lines of the file:
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@@
 <wire x1="10.668" y1="14.6304" x2="10.668" y2="14.9352" width="0.254" layer="16"/>
 <wire x1="17.6784" y1="29.5656" x2="19.2024" y2="31.0896" width="0.254" layer="16"/>
-<wire x1="4.8768" y1="25.908" x2="10.1208" y2="26.008" width="0.254" layer="16"/>
 <wire x1="19.2024" y1="31.0896" x2="19.2737" y2="31.1171" width="0.254" layer="16"/>
-<wire x1="4.8768" y1="25.908" x2="4.745" y2="25.81" width="0.254" layer="16"/>
 <wire x1="31.3944" y1="29.5656" x2="34.7472" y2="26.2128" width="0.254" layer="16"/>
 <wire x1="17.6784" y1="29.5656" x2="31.3944" y2="29.5656" width="0.254" layer="16"/>
@@
 <via x="16.764" y="13.1064" extent="1-16" drill="0.6096"/>
 <via x="10.668" y="14.9352" extent="1-16" drill="0.6096"/>
+<via x="9.9" y="25.2" extent="1-16" drill="0.5"/>
+<via x="9.9" y="21.6" extent="1-16" drill="0.5"/>
+<wire x1="9.9" y1="25.2" x2="9.9" y2="21.6" width="0.4064" layer="1"/>
 </signal>
 <signal name="TONE">

Commit message: update circuit, logo
Parts:
- R4: value 100k -> 90k
- moved LED1 0.17 mm to (8.28, 29.4), turned to 0 degrees
Routing:
- net N$1: track 8.54 -> 2.80 mm
- net INDICATOR: track 30.2 -> 33.5 mm
Other:
- board text added: "/Users/rmd/Downloads/flappy.bmp"
- board text removed: "/Users/rdiamond/Documents/flappy.bmp"

Commit message: logo
Routing:
- net 5V: track 167.8 -> 166.6 mm
- net SCK: track 8.80 -> 8.14 mm
Changed lines of the file:
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@@
 <wire x1="35.052" y1="28.6512" x2="34.99" y2="28.72" width="0.254" layer="1"/>
 <wire x1="17.6784" y1="34.7472" x2="14.3256" y2="31.3944" width="0.254" layer="1"/>
-<wire x1="30.1752" y1="34.7472" x2="17.6784" y2="34.7472" width="0.254" layer="1"/>
-<wire x1="30.1752" y1="28.6512" x2="30.1752" y2="34.7472" width="0.254" layer="1"/>
+<wire x1="30.1752" y1="32.6136" x2="28.2702" y2="34.7472" width="0.254" layer="1"/>
+<wire x1="28.2702" y1="34.7472" x2="17.6784" y2="34.7472" width="0.254" layer="1"/>
+<wire x1="30.1752" y1="28.6512" x2="30.1752" y2="32.6136" width="0.254" layer="1"/>
 <wire x1="30.1752" y1="28.6512" x2="30.41" y2="28.61" width="0.254" layer="1"/>
 <via x="7.62" y="13.4112" extent="1-16" drill="0.6096"/>
@@
 <contactref element="PROGRAMMING_HEADER" pad="3"/>
 <contactref element="U1" pad="9"/>
-<wire x1="23.1648" y1="11.5824" x2="25.2984" y2="11.5824" width="0.254" layer="1"/>
-<wire x1="23.1648" y1="5.4864" x2="23.1648" y2="11.5824" width="0.254" layer="1"/>
+<wire x1="24.257" y1="11.5824" x2="25.2984" y2="11.5824" width="0.254" layer="1"/>
+<wire x1="23.1648" y1="5.4864" x2="23.5458" y2="5.969" width="0.254" layer="1"/>
+<wire x1="23.5458" y1="5.969" x2="23.5458" y2="10.8966" width="0.254" layer="1"/>
+<wire x1="23.5458" y1="10.8966" x2="24.257" y2="11.5824" width="0.254" layer="1"/>
 <wire x1="25.2984" y1="11.5824" x2="25.5238" y2="11.66" width="0.254" layer="1"/>
 <wire x1="23.1648" y1="5.4864" x2="22.96" y2="5.225" width="0.254" layer="1"/>

Commit message: 0603 and gnd
Parts:
- C5, C6: device rcl:C0805 -> rcl:C0603
- R1, R2, R4, R5: device rcl:R0805 -> rcl:R0603
- moved PROGRAMMING_HEADER 1.39 mm to (23.2, 5.33)
Routing:
- net GND: track 132.6 -> 170.8 mm, vias 4 -> 8
- net TONE: track 51.0 -> 25.1 mm, vias 1 -> 0
- net MAGNETIC_SENSOR: track 28.7 -> 19.2 mm, vias 3 -> 2
- net N$5: track 22.6 -> 15.5 mm
- net LID_SERVO: track 35.2 -> 41.1 mm
- net ROLL_SERVO: track 18.1 -> 21.5 mm
- net INDICATOR: track 33.5 -> 35.3 mm
- net SCK: track 8.14 -> 6.65 mm
- net START_BUTTON: track 25.1 -> 23.6 mm
- net MISO: track 5.24 -> 3.89 mm
- net 5V: track 166.6 -> 165.3 mm
- net MOSI: track 8.75 -> 7.48 mm
- net RESET: track 12.0 -> 10.8 mm
- net USB_5V: track 27.1 -> 27.8 mm
- net CHARACTER_SERVO: track 16.8 -> 17.5 mm
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