File: circuit/bird.brd (EAGLE design)
At the start: 42.1 x 37.9 mm, 25 parts, among them J1 22-27-2031-03, U1 ATTINY84-20SSU, X1 MINI-USB-32005-201

Commit message: update board
Parts:
- removed S1: TL32PO, switch:TL3XPO
- C1: device rcl:C1206 -> rcl:C0603
- C2, C3, C4: device rcl:C1210 -> rcl:C0805
- R3: device rcl:R0805 -> rcl:R0603
Connections:
- removed net USB_5V: S1.1, X1.1
- net 5V: now also X1.1; no longer S1.2
Routing:
- net GND: track 170.8 -> 51.8 mm, vias 8 -> 6
- net USB_5V: track 27.8 -> 0.00 mm
- net LID_SERVO: track 41.1 -> 31.2 mm, vias 1 -> 2
- net N$5: track 15.5 -> 10.8 mm, vias 3 -> 2
- net 5V: track 165.3 -> 162.5 mm, vias 1 -> 0
- net INDICATOR: track 35.3 -> 37.9 mm
- net ROLL_SERVO: track 21.5 -> 23.7 mm
- net TONE: track 25.1 -> 26.7 mm, vias 0 -> 2
- net RESET: track 10.8 -> 9.34 mm, vias 1 -> 0
- net MAGNETIC_SENSOR: track 19.2 -> 20.5 mm
- net MAGNETIC_SENSOR_IN: track 5.40 -> 6.30 mm, vias 1 -> 0

Commit message: update board
Routing:
- net 5V: track 162.5 -> 161.3 mm
- net MAGNETIC_SENSOR_IN: track 6.30 -> 5.42 mm
Changed lines of the file:
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@@
 <wire x1="36.8808" y1="31.6992" x2="36.8808" y2="30.7848" width="0.254" layer="1"/>
 <wire x1="35.3568" y1="33.2232" x2="36.8808" y2="31.6992" width="0.254" layer="1"/>
-<wire x1="5.1816" y1="33.2232" x2="35.3568" y2="33.2232" width="0.254" layer="1"/>
-<wire x1="5.1816" y1="28.3464" x2="5.1816" y2="33.2232" width="0.254" layer="1"/>
+<wire x1="7.4168" y1="33.2232" x2="35.3568" y2="33.2232" width="0.254" layer="1"/>
+<wire x1="5.1816" y1="28.3464" x2="5.1816" y2="31.0896" width="0.254" layer="1"/>
+<wire x1="5.1816" y1="31.0896" x2="7.3152" y2="33.2232" width="0.254" layer="1"/>
+<wire x1="7.3152" y1="33.2232" x2="7.4168" y2="33.2232" width="0.254" layer="1"/>
 <wire x1="11.5824" y1="21.9456" x2="5.1816" y2="28.3464" width="0.254" layer="1"/>
 <wire x1="35.052" y1="28.956" x2="34.99" y2="28.72" width="0.254" layer="1"/>
@@
 <contactref element="J1" pad="3"/>
 <contactref element="R2" pad="1"/>
-<wire x1="4.8768" y1="19.5072" x2="9.144" y2="19.5072" width="0.254" layer="1"/>
-<wire x1="4.8768" y1="17.9832" x2="4.8768" y2="19.5072" width="0.254" layer="1"/>
+<wire x1="6.35" y1="19.5072" x2="9.144" y2="19.5072" width="0.254" layer="1"/>
+<wire x1="4.8768" y1="17.9832" x2="6.35" y2="19.5072" width="0.254" layer="1"/>
 <wire x1="9.144" y1="19.5072" x2="9.2172" y2="19.719" width="0.254" layer="1"/>
 <wire x1="4.8768" y1="17.9832" x2="4.845" y2="17.705" width="0.254" layer="1"/>
