File: circuit/bird.sch (EAGLE design)
At the start: 15 parts, among them J1 22-27-2031-03, U1 ATTINY84-20SSU

Commit message: update sensor
Parts:
- added R2, R3: 10k 1%, rcl:R-US_R0603
Connections:
- new net MAGNETIC_REFERENCE: R2.2, R3.1, U1.PA3
- net 5V: now also R2.1
- net GND: now also R3.2
Changed lines of the file:
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@@
 <part name="R1" library="rcl" deviceset="R-US_" device="R1206" value="500"/>
 <part name="P+1" library="supply1" deviceset="+5V" device=""/>
+<part name="R2" library="rcl" deviceset="R-US_" device="R0603" value="10k 1%"/>
+<part name="R3" library="rcl" deviceset="R-US_" device="R0603" value="10k 1%"/>
+<part name="U$5" library="SparkFun" deviceset="5V" device=""/>
+<part name="GND8" library="SparkFun" deviceset="GND" device=""/>
 <part name="J1" library="con-molex" deviceset="22-?-03" device="27-2031"/>
 <part name="U$6" library="SparkFun" deviceset="5V" device=""/>
@@
 <instance part="R1" gate="G$1" x="68.58" y="50.8" rot="R90"/>
 <instance part="P+1" gate="1" x="68.58" y="63.5"/>
+<instance part="R2" gate="G$1" x="-20.32" y="-10.16"/>
+<instance part="R3" gate="G$1" x="-5.08" y="-10.16"/>
+<instance part="U$5" gate="G$1" x="-30.48" y="-2.54"/>
+<instance part="GND8" gate="1" x="7.62" y="-20.32"/>
 <instance part="J1" gate="-1" x="121.92" y="-5.08"/>
 <instance part="J1" gate="-2" x="121.92" y="-10.16"/>
@@
 </segment>
 <segment>
+<pinref part="R2" gate="G$1" pin="1"/>
+<wire x1="-25.4" y1="-10.16" x2="-30.48" y2="-10.16" width="0.1524" layer="91"/>
+<wire x1="-30.48" y1="-10.16" x2="-30.48" y2="-2.54" width="0.1524" layer="91"/>
+<pinref part="U$5" gate="G$1" pin="5V"/>
+</segment>
+<segment>
 <pinref part="J1" gate="-1" pin="S"/>
 <wire x1="119.38" y1="-5.08" x2="91.44" y2="-5.08" width="0.1524" layer="91"/>
@@
 </segment>
 <segment>
+<pinref part="R3" gate="G$1" pin="2"/>
+<wire x1="0" y1="-10.16" x2="7.62" y2="-10.16" width="0.1524" layer="91"/>
+<wire x1="7.62" y1="-10.16" x2="7.62" y2="-17.78" width="0.1524" layer="91"/>
+<pinref part="GND8" gate="1" pin="GND"/>
+</segment>
+<segment>
 <pinref part="J1" gate="-2" pin="S"/>
 <wire x1="119.38" y1="-10.16" x2="93.98" y2="-10.16" width="0.1524" layer="91"/>
@@
 </segment>
 </net>
+<net name="MAGNETIC_REFERENCE" class="0">
+<segment>
+<pinref part="U1" gate="A" pin="PA3"/>
+<wire x1="20.32" y1="40.64" x2="38.1" y2="40.64" width="0.1524" layer="91"/>
+<label x="22.86" y="40.64" size="1.778" layer="95"/>
+</segment>
+<segment>
+<pinref part="R2" gate="G$1" pin="2"/>
+<pinref part="R3" gate="G$1" pin="1"/>
+<wire x1="-15.24" y1="-10.16" x2="-12.7" y2="-10.16" width="0.1524" layer="91"/>
+<wire x1="-12.7" y1="-10.16" x2="-10.16" y2="-10.16" width="0.1524" layer="91"/>
+<wire x1="-12.7" y1="-10.16" x2="-12.7" y2="2.54" width="0.1524" layer="91"/>
+<junction x="-12.7" y="-10.16"/>
+<wire x1="-12.7" y1="2.54" x2="10.16" y2="2.54" width="0.1524" layer="91"/>
+<label x="-10.16" y="2.54" size="1.778" layer="95"/>
+</segment>
+</net>

Commit message: use constants
Parts:
- removed R2, R3: 10k 1%, rcl:R-US_R0603
Connections:
- net 5V: no longer R2.1
- net GND: no longer R3.2
- net MAGNETIC_REFERENCE: no longer R2.2, R3.1
Changed lines of the file:
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@@
 <part name="R1" library="rcl" deviceset="R-US_" device="R1206" value="500"/>
 <part name="P+1" library="supply1" deviceset="+5V" device=""/>
-<part name="R2" library="rcl" deviceset="R-US_" device="R0603" value="10k 1%"/>
-<part name="R3" library="rcl" deviceset="R-US_" device="R0603" value="10k 1%"/>
-<part name="U$5" library="SparkFun" deviceset="5V" device=""/>
-<part name="GND8" library="SparkFun" deviceset="GND" device=""/>
 <part name="J1" library="con-molex" deviceset="22-?-03" device="27-2031"/>
 <part name="U$6" library="SparkFun" deviceset="5V" device=""/>
@@
 <instance part="R1" gate="G$1" x="68.58" y="50.8" rot="R90"/>
 <instance part="P+1" gate="1" x="68.58" y="63.5"/>
-<instance part="R2" gate="G$1" x="-20.32" y="-10.16"/>
-<instance part="R3" gate="G$1" x="-5.08" y="-10.16"/>
-<instance part="U$5" gate="G$1" x="-30.48" y="-2.54"/>
-<instance part="GND8" gate="1" x="7.62" y="-20.32"/>
 <instance part="J1" gate="-1" x="121.92" y="-5.08"/>
 <instance part="J1" gate="-2" x="121.92" y="-10.16"/>
@@
 </segment>
 <segment>
-<pinref part="R2" gate="G$1" pin="1"/>
-<wire x1="-25.4" y1="-10.16" x2="-30.48" y2="-10.16" width="0.1524" layer="91"/>
-<wire x1="-30.48" y1="-10.16" x2="-30.48" y2="-2.54" width="0.1524" layer="91"/>
-<pinref part="U$5" gate="G$1" pin="5V"/>
-</segment>
-<segment>
 <pinref part="J1" gate="-1" pin="S"/>
 <wire x1="119.38" y1="-5.08" x2="91.44" y2="-5.08" width="0.1524" layer="91"/>
@@
 </segment>
 <segment>
-<pinref part="R3" gate="G$1" pin="2"/>
-<wire x1="0" y1="-10.16" x2="7.62" y2="-10.16" width="0.1524" layer="91"/>
-<wire x1="7.62" y1="-10.16" x2="7.62" y2="-17.78" width="0.1524" layer="91"/>
-<pinref part="GND8" gate="1" pin="GND"/>
-</segment>
-<segment>
 <pinref part="J1" gate="-2" pin="S"/>
 <wire x1="119.38" y1="-10.16" x2="93.98" y2="-10.16" width="0.1524" layer="91"/>
@@
 <label x="22.86" y="40.64" size="1.778" layer="95"/>
 </segment>
-<segment>
-<pinref part="R2" gate="G$1" pin="2"/>
-<pinref part="R3" gate="G$1" pin="1"/>
-<wire x1="-15.24" y1="-10.16" x2="-12.7" y2="-10.16" width="0.1524" layer="91"/>
-<wire x1="-12.7" y1="-10.16" x2="-10.16" y2="-10.16" width="0.1524" layer="91"/>
-<wire x1="-12.7" y1="-10.16" x2="-12.7" y2="2.54" width="0.1524" layer="91"/>
-<junction x="-12.7" y="-10.16"/>
-<wire x1="-12.7" y1="2.54" x2="10.16" y2="2.54" width="0.1524" layer="91"/>
-<label x="-10.16" y="2.54" size="1.778" layer="95"/>
-</segment>
-</net>
+</net>

Commit message: new layout
Parts:
- removed SPEAKER: 22-27-2021-02, con-molex:22-27-2021-02
- added C5: 220pf, rcl:C-USC0805
- added C6: .01uf, rcl:C-USC0805
- added C7: 10uf, rcl:C-USC0805
- added R2: 47k, rcl:R-US_R0805
- added R3: 10M, rcl:R-US_R0805
- added R4, R5: 100k, rcl:R-US_R0805
- added S1: TL32PO, switch:TL32PO
- added SG2: F/QMX, buzzer:F/QMX
- added U$5: MCP601, SparkFun:MCP601
- C2, C3, C4: value (none) -> 10u
- LED1: device led:LED5MM -> led:LEDSML1206
- R1: device rcl:R-US_R1206 -> rcl:R-US_R0805
Connections:
- new net MAGNETIC_SENSOR_IN: J1-3.S, R2.1
- new net N$2: C1.1, POWER_IN-2.S, S1.O
- new net N$4: C5.1, R2.2, R3.2, U$5.V-
- new net N$5: R4.1, R5.2, U$5.V+
- net 5V: now also C6.1, C7.1, R4.2, S1.P, U$5.VDD; no longer C1.1, POWER_IN-2.S
- net GND: now also C6.2, C7.2, R5.1, SG2.1, U$5.VSS; no longer SPEAKER-2.S
- net MAGNETIC_SENSOR: now also C5.2, R3.1, U$5.VOUT; no longer J1-3.S
- net TONE: now also SG2.2; no longer SPEAKER-1.S
Other:
- note added: "CPU"
- note added: "Connectors"
- note added: "Inverting Amplifier"
- note added: "Linear Hall Effect Sensor"
- note added: "Low pass filter"
- note added: "Voltage Divider Provides reference voltage"

Commit message: usb
Parts:
- removed POWER_IN: 22-27-2021-02, con-molex:22-27-2021-02
- added X1: MINI-USB-32005-201, con-cypressindustries:MINI-USB-32005-201
Connections:
- removed net N$2: C1.1, POWER_IN-2.S, S1.O
- new net D+: X1.3
- new net D-: X1.2
- new net USB_5V: S1.O, X1.1
- net 5V: now also C1.1
- net GND: now also X1.5; no longer POWER_IN-1.S

Commit message: cleanups and fix sketch
Parts:
- added TP1: TEST-POINT2, SparkFun:TEST-POINT2
Connections:
- net MAGNETIC_REFERENCE: now also TP1.1
Changed lines of the file:
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@@
 <part name="X1" library="con-cypressindustries" deviceset="MINI-USB-" device="32005-201"/>
 <part name="GND8" library="SparkFun-Aesthetics" deviceset="GND" device=""/>
+<part name="TP1" library="SparkFun" deviceset="TEST-POINT" device="2"/>
 </parts>
 <sheets>
@@
 <instance part="X1" gate="G$1" x="-114.3" y="-20.32" rot="R180"/>
 <instance part="GND8" gate="1" x="-134.62" y="-20.32"/>
+<instance part="TP1" gate="G$1" x="50.8" y="45.72"/>
 </instances>
 <busses>
@@
 <wire x1="20.32" y1="40.64" x2="38.1" y2="40.64" width="0.1524" layer="91"/>
 <label x="22.86" y="40.64" size="1.778" layer="95"/>
-</segment>
-</net>
+<pinref part="TP1" gate="G$1" pin="1"/>
+<wire x1="38.1" y1="40.64" x2="50.8" y2="40.64" width="0.1524" layer="91"/>
+<wire x1="50.8" y1="40.64" x2="50.8" y2="45.72" width="0.1524" layer="91"/>
+</segment>
+</net>

Commit message: update circuit, logo
Parts:
- R4: value 100k -> 90k
Changed lines of the file:
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@@
 <part name="R2" library="rcl" deviceset="R-US_" device="R0805" value="47k"/>
 <part name="R3" library="rcl" deviceset="R-US_" device="R0805" value="10M"/>
-<part name="R4" library="rcl" deviceset="R-US_" device="R0805" value="100k"/>
+<part name="R4" library="rcl" deviceset="R-US_" device="R0805" value="90k"/>
 <part name="R5" library="rcl" deviceset="R-US_" device="R0805" value="100k"/>
 <part name="C5" library="rcl" deviceset="C-US" device="C0805" value="220pf"/>

Commit message: 0603 and gnd
Parts:
- C5, C6: device rcl:C-USC0805 -> rcl:C-USC0603
- R1, R2, R4, R5: device rcl:R-US_R0805 -> rcl:R-US_R0603
Changed lines of the file:
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@@
 <grid distance="0.1" unitdist="inch" unit="inch" style="lines" multiple="1" display="no" altdistance="0.01" altunitdist="inch" altunit="inch"/>
 <layers>
-<layer number="1" name="Top" color="4" fill="1" visible="no" active="no"/>
-<layer number="2" name="Route2" color="1" fill="3" visible="no" active="no"/>
-<layer number="3" name="Route3" color="4" fill="3" visible="no" active="no"/>
-<layer number="14" name="Route14" color="1" fill="6" visible="no" active="no"/>
-<layer number="15" name="Route15" color="4" fill="6" visible="no" active="no"/>
-<layer number="16" name="Bottom" color="1" fill="1" visible="no" active="no"/>
-<layer number="17" name="Pads" color="2" fill="1" visible="no" active="no"/>
-<layer number="18" name="Vias" color="2" fill="1" visible="no" active="no"/>
-<layer number="19" name="Unrouted" color="6" fill="1" visible="no" active="no"/>
-<layer number="20" name="Dimension" color="15" fill="1" visible="no" active="no"/>
-<layer number="21" name="tPlace" color="7" fill="1" visible="no" active="no"/>
-<layer number="22" name="bPlace" color="7" fill="1" visible="no" active="no"/>
-<layer number="23" name="tOrigins" color="15" fill="1" visible="no" active="no"/>
-<layer number="24" name="bOrigins" color="15" fill="1" visible="no" active="no"/>
-<layer number="25" name="tNames" color="7" fill="1" visible="no" active="no"/>
-<layer number="26" name="bNames" color="7" fill="1" visible="no" active="no"/>
-<layer number="27" name="tValues" color="7" fill="1" visible="no" active="no"/>
-<layer number="28" name="bValues" color="7" fill="1" visible="no" active="no"/>
+<layer number="1" name="Top" color="4" fill="1" visible="yes" active="no"/>
+<layer number="2" name="Route2" color="1" fill="3" visible="yes" active="no"/>
+<layer number="3" name="Route3" color="4" fill="3" visible="yes" active="no"/>
+<layer number="14" name="Route14" color="1" fill="6" visible="yes" active="no"/>
+<layer number="15" name="Route15" color="4" fill="6" visible="yes" active="no"/>
+<layer number="16" name="Bottom" color="1" fill="1" visible="yes" active="no"/>
+<layer number="17" name="Pads" color="2" fill="1" visible="yes" active="no"/>
+<layer number="18" name="Vias" color="2" fill="1" visible="yes" active="no"/>
+<layer number="19" name="Unrouted" color="6" fill="1" visible="yes" active="no"/>
+<layer number="20" name="Dimension" color="15" fill="1" visible="yes" active="no"/>
+<layer number="21" name="tPlace" color="7" fill="1" visible="yes" active="no"/>
+<layer number="22" name="bPlace" color="7" fill="1" visible="yes" active="no"/>
+<layer number="23" name="tOrigins" color="15" fill="1" visible="yes" active="no"/>
+<layer number="24" name="bOrigins" color="15" fill="1" visible="yes" active="no"/>
+<layer number="25" name="tNames" color="7" fill="1" visible="yes" active="no"/>
+<layer number="26" name="bNames" color="7" fill="1" visible="yes" active="no"/>
+<layer number="27" name="tValues" color="7" fill="1" visible="yes" active="no"/>
+<layer number="28" name="bValues" color="7" fill="1" visible="yes" active="no"/>
 <layer number="29" name="tStop" color="7" fill="3" visible="no" active="no"/>
 <layer number="30" name="bStop" color="7" fill="6" visible="no" active="no"/>
@@
 <layer number="35" name="tGlue" color="7" fill="4" visible="no" active="no"/>
 <layer number="36" name="bGlue" color="7" fill="5" visible="no" active="no"/>
-<layer number="37" name="tTest" color="7" fill="1" visible="no" active="no"/>
-<layer number="38" name="bTest" color="7" fill="1" visible="no" active="no"/>
+<layer number="37" name="tTest" color="7" fill="1" visible="yes" active="no"/>
+<layer number="38" name="bTest" color="7" fill="1" visible="yes" active="no"/>
 <layer number="39" name="tKeepout" color="4" fill="11" visible="no" active="no"/>
 <layer number="40" name="bKeepout" color="1" fill="11" visible="no" active="no"/>
@@
 <layer number="44" name="Drills" color="7" fill="1" visible="no" active="no"/>
 <layer number="45" name="Holes" color="7" fill="1" visible="no" active="no"/>
-<layer number="46" name="Milling" color="3" fill="1" visible="no" active="no"/>
-<layer number="47" name="Measures" color="7" fill="1" visible="no" active="no"/>
-<layer number="48" name="Document" color="7" fill="1" visible="no" active="no"/>
-<layer number="49" name="Reference" color="7" fill="1" visible="no" active="no"/>
-<layer number="50" name="dxf" color="7" fill="1" visible="no" active="no"/>
-<layer number="51" name="tDocu" color="7" fill="1" visible="no" active="no"/>
-<layer number="52" name="bDocu" color="7" fill="1" visible="no" active="no"/>
-<layer number="53" name="tGND_GNDA" color="7" fill="9" visible="no" active="no"/>
-<layer number="54" name="bGND_GNDA" color="1" fill="9" visible="no" active="no"/>
-<layer number="56" name="wert" color="7" fill="1" visible="no" active="no"/>
+<layer number="46" name="Milling" color="3" fill="1" visible="yes" active="no"/>
+<layer number="47" name="Measures" color="7" fill="1" visible="yes" active="no"/>
+<layer number="48" name="Document" color="7" fill="1" visible="yes" active="no"/>
+<layer number="49" name="Reference" color="7" fill="1" visible="yes" active="no"/>
+<layer number="50" name="dxf" color="7" fill="1" visible="yes" active="no"/>
+<layer number="51" name="tDocu" color="7" fill="1" visible="yes" active="no"/>
+<layer number="52" name="bDocu" color="7" fill="1" visible="yes" active="no"/>
+<layer number="53" name="tGND_GNDA" color="7" fill="9" visible="yes" active="no"/>
+<layer number="54" name="bGND_GNDA" color="1" fill="9" visible="yes" active="no"/>
+<layer number="56" name="wert" color="7" fill="1" visible="yes" active="no"/>
 <layer number="91" name="Nets" color="2" fill="1" visible="yes" active="yes"/>
 <layer number="92" name="Busses" color="1" fill="1" visible="yes" active="yes"/>
@@
 <part name="PROGRAMMING_HEADER" library="pinhead" deviceset="PINHD-2X3" device=""/>
 <part name="LED1" library="led" deviceset="LED" device="SML1206" value="red"/>
-<part name="R1" library="rcl" deviceset="R-US_" device="R0805" value="500"/>
+<part name="R1" library="rcl" deviceset="R-US_" device="R0603" value="500"/>
 <part name="P+1" library="supply1" deviceset="+5V" device=""/>
 <part name="J1" library="con-molex" deviceset="22-?-03" device="27-2031"/>
@@
 <part name="U$8" library="SparkFun" deviceset="5V" device=""/>
 <part name="GND10" library="SparkFun" deviceset="GND" device=""/>
-<part name="R2" library="rcl" deviceset="R-US_" device="R0805" value="47k"/>
+<part name="R2" library="rcl" deviceset="R-US_" device="R0603" value="47k"/>
 <part name="R3" library="rcl" deviceset="R-US_" device="R0805" value="10M"/>
-<part name="R4" library="rcl" deviceset="R-US_" device="R0805" value="90k"/>
-<part name="R5" library="rcl" deviceset="R-US_" device="R0805" value="100k"/>
-<part name="C5" library="rcl" deviceset="C-US" device="C0805" value="220pf"/>
-<part name="C6" library="rcl" deviceset="C-US" device="C0805" value=".01uf"/>
+<part name="R4" library="rcl" deviceset="R-US_" device="R0603" value="90k"/>
+<part name="R5" library="rcl" deviceset="R-US_" device="R0603" value="100k"/>
+<part name="C5" library="rcl" deviceset="C-US" device="C0603" value="220pf"/>
+<part name="C6" library="rcl" deviceset="C-US" device="C0603" value=".01uf"/>
 <part name="C7" library="rcl" deviceset="C-US" device="C0805" value="10uf"/>
 <part name="U$10" library="SparkFun" deviceset="5V" device=""/>

Commit message: update board
Parts:
- removed S1: TL32PO, switch:TL32PO
- C1: device rcl:C-USC1206 -> rcl:C-USC0603
- C2, C3, C4: device rcl:C-USC1210 -> rcl:C-USC0805
- R3: device rcl:R-US_R0805 -> rcl:R-US_R0603
Connections:
- removed net USB_5V: S1.O, X1.1
- net 5V: now also X1.1; no longer S1.P
Changed lines of the file:
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@@
 <part name="ROLLING_SERVO" library="con-molex" deviceset="22-?-03" device="27-2031"/>
 <part name="START_BUTTON" library="con-molex" deviceset="22-?-02" device="27-2021"/>
-<part name="C1" library="rcl" deviceset="C-US" device="C1206" value=".1uF"/>
+<part name="C1" library="rcl" deviceset="C-US" device="C0603" value=".1uF"/>
 <part name="U$1" library="SparkFun" deviceset="5V" device="" value="4.5V"/>
 <part name="GND1" library="SparkFun" deviceset="GND" device=""/>
@@
 <part name="U$6" library="SparkFun" deviceset="5V" device=""/>
 <part name="GND6" library="SparkFun" deviceset="GND" device=""/>
-<part name="C2" library="rcl" deviceset="C-US" device="C1210" value="10u"/>
-<part name="C3" library="rcl" deviceset="C-US" device="C1210" value="10u"/>
-<part name="C4" library="rcl" deviceset="C-US" device="C1210" value="10u"/>
+<part name="C2" library="rcl" deviceset="C-US" device="C0805" value="10u"/>
+<part name="C3" library="rcl" deviceset="C-US" device="C0805" value="10u"/>
+<part name="C4" library="rcl" deviceset="C-US" device="C0805" value="10u"/>
 <part name="SUPPLY1" library="SparkFun-Aesthetics" deviceset="5V" device=""/>
 <part name="GND9" library="SparkFun-Aesthetics" deviceset="GND" device=""/>
@@
 <part name="GND10" library="SparkFun" deviceset="GND" device=""/>
 <part name="R2" library="rcl" deviceset="R-US_" device="R0603" value="47k"/>
-<part name="R3" library="rcl" deviceset="R-US_" device="R0805" value="10M"/>
+<part name="R3" library="rcl" deviceset="R-US_" device="R0603" value="10M"/>
 <part name="R4" library="rcl" deviceset="R-US_" device="R0603" value="90k"/>
 <part name="R5" library="rcl" deviceset="R-US_" device="R0603" value="100k"/>
@@
 <part name="GND13" library="SparkFun" deviceset="GND" device=""/>
 <part name="SG2" library="buzzer" deviceset="F/QMX" device=""/>
-<part name="S1" library="switch" deviceset="TL32PO" device=""/>
 <part name="X1" library="con-cypressindustries" deviceset="MINI-USB-" device="32005-201"/>
 <part name="GND8" library="SparkFun-Aesthetics" deviceset="GND" device=""/>
@@
 <instance part="GND13" gate="1" x="-185.42" y="60.96"/>
 <instance part="SG2" gate="G$1" x="127" y="-35.56" rot="MR90"/>
-<instance part="S1" gate="BEF1" x="-33.02" y="58.42" rot="R90"/>
 <instance part="X1" gate="G$1" x="-114.3" y="-20.32" rot="R180"/>
 <instance part="GND8" gate="1" x="-134.62" y="-20.32"/>
@@
 <wire x1="-20.32" y1="53.34" x2="-20.32" y2="48.26" width="0.1524" layer="91"/>
 <wire x1="-20.32" y1="48.26" x2="-15.24" y2="48.26" width="0.1524" layer="91"/>
-<wire x1="-27.94" y1="58.42" x2="-25.4" y2="58.42" width="0.1524" layer="91"/>
-<wire x1="-25.4" y1="58.42" x2="-25.4" y2="50.8" width="0.1524" layer="91"/>
+<wire x1="-25.4" y1="53.34" x2="-25.4" y2="50.8" width="0.1524" layer="91"/>
 <wire x1="-25.4" y1="50.8" x2="-25.4" y2="48.26" width="0.1524" layer="91"/>
 <wire x1="-25.4" y1="48.26" x2="-20.32" y2="48.26" width="0.1524" layer="91"/>
 <junction x="-20.32" y="48.26"/>
-<pinref part="S1" gate="BEF1" pin="P"/>
 <pinref part="C1" gate="G$1" pin="1"/>
 <wire x1="-45.72" y1="50.8" x2="-25.4" y2="50.8" width="0.1524" layer="91"/>
 <junction x="-25.4" y="50.8"/>
+<wire x1="-55.88" y1="53.34" x2="-45.72" y2="53.34" width="0.1524" layer="91"/>
+<wire x1="-27.94" y1="53.34" x2="-40.64" y2="53.34" width="0.1524" layer="91"/>
+<wire x1="-40.64" y1="53.34" x2="-45.72" y2="53.34" width="0.1524" layer="91"/>
+<label x="-55.88" y="53.34" size="1.778" layer="95"/>
+<wire x1="-27.94" y1="53.34" x2="-25.4" y2="53.34" width="0.1524" layer="91"/>
 </segment>
 <segment>
@@
 <wire x1="-198.12" y1="30.48" x2="-198.12" y2="27.94" width="0.1524" layer="91"/>
 <junction x="-203.2" y="30.48"/>
+</segment>
+<segment>
+<pinref part="X1" gate="G$1" pin="1"/>
+<wire x1="-109.22" y1="-25.4" x2="-73.66" y2="-25.4" width="0.1524" layer="91"/>
+<label x="-83.82" y="-25.4" size="1.778" layer="95"/>
 </segment>
 </net>
@@
 </segment>
 </net>
-<net name="USB_5V" class="0">
-<segment>
-<pinref part="X1" gate="G$1" pin="1"/>
-<wire x1="-109.22" y1="-25.4" x2="-73.66" y2="-25.4" width="0.1524" layer="91"/>
-<label x="-83.82" y="-25.4" size="1.778" layer="95"/>
-</segment>
-<segment>
-<wire x1="-55.88" y1="53.34" x2="-45.72" y2="53.34" width="0.1524" layer="91"/>
-<wire x1="-38.1" y1="55.88" x2="-40.64" y2="55.88" width="0.1524" layer="91"/>
-<wire x1="-40.64" y1="55.88" x2="-40.64" y2="53.34" width="0.1524" layer="91"/>
-<wire x1="-40.64" y1="53.34" x2="-45.72" y2="53.34" width="0.1524" layer="91"/>
-<pinref part="S1" gate="BEF1" pin="O"/>
-<label x="-55.88" y="53.34" size="1.778" layer="95"/>
-</segment>
-</net>
